File: SFD/Hardware/RJ45/SFD_N.brd (EAGLE design)
At the start: 77 x 85 mm, 32 parts, among them IC1 78L05, IC2 ATtiny2313, IC3 LM393N, IC4 ULN 2803A, IC5 ULN 2803A, T1 BC557, T2 BC547, X1 RJ45 8P8C, X2 RJ45 8P8C

Commit message: Update
Connections:
- net GND: now also IC2.4, IC2.5
Routing:
- net GND: track 271.8 -> 277.0 mm
Other:
- board text added: "Rev 1.1"
- board text added: "© S. Marsch SFD_N"
- board text removed: "© S. Marsch SFD-V1-N"
Changed lines of the file:
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@@
 <wire x1="0" y1="85" x2="0" y2="0" width="0" layer="20"/>
 <text x="2.667" y="9.271" size="1.778" layer="25">© S. Marsch
- SFD-V1-N</text>
+   SFD_N</text>
+<text x="4.699" y="1.143" size="1.778" layer="25">Rev 1.1</text>
 </plain>
 <attributes>
@@
 </element>
 <element name="LED1" library="led" package="LED3MM" value="Rot" x="9.017" y="6.096" smashed="yes">
-<attribute name="NAME" x="12.192" y="5.207" size="1.27" layer="25" ratio="10"/>
-<attribute name="VALUE" x="10.922" y="4.445" size="1.27" layer="27" ratio="10"/>
+<attribute name="NAME" x="11.811" y="5.588" size="1.27" layer="25" ratio="10"/>
+<attribute name="VALUE" x="3.302" y="5.715" size="1.27" layer="27" ratio="10"/>
 </element>
 <element name="R1" library="rcl" package="0207/10" value="27k" x="59.182" y="23.241" smashed="yes">
@@
 <wire x1="52.3494" y1="32.9184" x2="52.324" y2="32.893" width="0.254" layer="16"/>
 <wire x1="56.007" y1="35.2044" x2="56.007" y2="35.306" width="0.254" layer="16"/>
-<wire x1="5.207" y1="35.306" x2="30.734" y2="35.306" width="0.254" layer="16"/>
+<wire x1="5.207" y1="35.306" x2="16.51" y2="35.306" width="0.254" layer="16"/>
 <polygon width="0.254" layer="16" isolate="0.4064">
 <vertex x="0" y="0"/>
@@
 <contactref element="X2" pad="6"/>
 <contactref element="X2" pad="4"/>
+<wire x1="16.51" y1="35.306" x2="19.05" y2="35.306" width="0.254" layer="16"/>
+<wire x1="19.05" y1="35.306" x2="30.734" y2="35.306" width="0.254" layer="16"/>
 <wire x1="31.877" y1="34.163" x2="30.734" y2="35.306" width="0.254" layer="16"/>
 <wire x1="61.2648" y1="9.3726" x2="59.436" y2="9.3726" width="0.508" layer="1"/>
@@
 <wire x1="68.993" y1="35.306" x2="59.182" y2="35.306" width="0.254" layer="16"/>
 <wire x1="59.182" y1="35.306" x2="56.007" y2="35.306" width="0.254" layer="16"/>
+<contactref element="IC2" pad="4"/>
+<contactref element="IC2" pad="5"/>
+<wire x1="16.637" y1="32.766" x2="16.51" y2="32.893" width="0.254" layer="16"/>
+<wire x1="16.51" y1="32.893" x2="16.51" y2="35.306" width="0.254" layer="16"/>
+<wire x1="19.177" y1="32.766" x2="19.05" y2="32.893" width="0.254" layer="16"/>
+<wire x1="19.05" y1="32.893" x2="19.05" y2="35.306" width="0.254" layer="16"/>
 </signal>
 <signal name="N$13">
